File: Circuit/KiCAD Circuit/MAX1758.kicad_sch (KiCad schematic)
At the start: 34 parts, among them U1 MAX1758, U2 ArduinoMKRZero, U3 MC7805ACTG

Commit message: Backup
Parts:
- renumbered C2 to C?, C4 to C?, C10 to C?, C1 to C?, C13 to C?, C17 to C?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
