File: Circuit/KiCAD Circuit/Powerbank.kicad_pcb (KiCad board)
At the start: 2 copper layers, 44 parts, among them J1 EBWA-04-A, Q1 NMOS, Q2 PMOS, Q3 NMOS, SW1 SW_Push, SW2 SW_SPST, U1 BQ7692003PW

Commit message: Backup
Parts:
- moved D3 137.9 mm to (101.0, 138.4)
- moved R1 108.7 mm to (119.1, 128.3), turned to 180 degrees
- moved R3 94.8 mm to (134.6, 128.3), turned to 180 degrees
- moved SW2 73.4 mm to (162.6, 71.6), turned to 90 degrees
- moved C7 72.4 mm to (153.7, 83.8), turned to -90 degrees
- moved C5 56.5 mm to (139.7, 71.1), turned to -90 degrees
- moved A1 51.9 mm to (138.4, 103.5), turned to -90 degrees
- moved C4 50.4 mm to (150.6, 79.4), turned to 180 degrees
- moved R6 46.8 mm to (135.9, 71.1), turned to -90 degrees
- moved SW1 40.8 mm to (117.7, 78.7)
- moved R5 37.4 mm to (124.5, 78.7)
- moved R4 35.1 mm to (143.9, 79.5), turned to 90 degrees
- moved C8 33.1 mm to (153.7, 141.0)
- moved C1 29.2 mm to (109.3, 105.4)
- moved C6 29.1 mm to (142.3, 141.0)
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Routing:
- net Net-(D1-A): track 98.9 -> 221.2 mm
- net Net-(U1-SRP): track 0.00 -> 62.1 mm
- net Net-(U1-SRN): track 0.00 -> 56.0 mm
- net Net-(Q1-G): track 0.00 -> 53.2 mm
- net Net-(SW2-A): track 0.00 -> 42.8 mm
- net Net-(A1-A5/SCL): track 0.00 -> 31.6 mm
- net Net-(U1-TS1): track 0.00 -> 30.8 mm
- net Net-(Q1-S): track 9.40 -> 35.3 mm
- net Net-(Q2-D): track 0.00 -> 22.8 mm
- net Net-(U1-ALERT): track 0.00 -> 21.3 mm
- net Net-(U1-VC1): track 23.3 -> 39.6 mm
- net Net-(Q3-S): track 15.2 -> 24.7 mm
- net Net-(C6-Pad2): track 0.00 -> 6.35 mm
- net Net-(Q1-D): track 11.4 -> 6.35 mm
- net Net-(U1-REGOUT): track 15.0 -> 10.1 mm
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- added copper zone on B.Cu, net GND
Other:
- board outline added: 96.5 x 99.1 mm

Commit message: Backup
Parts:
- added G1: LOGO, Symbol:Do Not Touch Symbol, F.Cu at (111.8, 118.4)
- added G2: OSHW-Logo_7.5x8mm_SilkScreen, Symbol:OSHW-Logo_7.5x8mm_SilkScreen, F.Cu at (102.9, 92.7)
- added NT1: NetTie, Custom Footprints:NetTie General Net Class, F.Cu at (109.7, 97.8)
- added NT2: NetTie, Custom Footprints:NetTie General Net Class, F.Cu at (139.7, 109.2)
- added REF1: KiCad-Logo2_5mm_SilkScreen, Symbol:KiCad-Logo2_5mm_SilkScreen, F.Cu at (171.2, 130.6)
- Q2: footprint VP3203N3-G:TO-92_MC_MCH -> Custom Footprints:TO-92_MC_MCH
- moved C4 39.6 mm to (140.0, 117.5), turned to 90 degrees
- moved R4 36.6 mm to (142.7, 116.1), turned to 0 degrees
- moved A1 32.5 mm to (166.4, 120.0), turned to 0 degrees
- moved Rd2 29.3 mm to (153.7, 79.8)
- moved Cf1 29.0 mm to (141.5, 100.3), turned to 90 degrees
- moved D2 28.8 mm to (151.1, 85.4)
- moved D1 28.8 mm to (142.2, 85.4)
- moved Rd1 28.8 mm to (146.1, 79.8)
- moved Rf1 24.3 mm to (144.8, 90.2)
- moved SW2 24.2 mm to (154.9, 94.6)
- moved C7 23.3 mm to (144.8, 105.4)
- moved C9 22.4 mm to (149.2, 102.9), turned to 0 degrees
- moved U1 21.7 mm to (138.4, 105.4)
- moved C5 21.4 mm to (126.1, 87.6)
- moved R6 20.8 mm to (123.2, 87.6)
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Connections:
- D3 pad 1: Net-(D1-A) -> Net-(D3-K)
- H1 pad 1: Net-(D1-A) -> Net-(D3-K)
- H7 pad 1: Net-(D1-A) -> Net-(D3-K)
- J1 pad 4: Net-(D1-A) -> Net-(D3-K)
- Rc1 pad 1: Net-(D1-A) -> Net-(D3-K)
- U1 pad 3: GND -> Net-(U1-VSS)
Routing:
- net Net-(D1-A): track 221.2 -> 55.3 mm
- net Net-(D3-K): track 0.00 -> 119.5 mm
- net Net-(A1-A4/SDA): track 0.00 -> 37.0 mm
- net Net-(U1-SRN): track 56.0 -> 22.9 mm
- net Net-(U1-SRP): track 62.1 -> 30.9 mm
- net Net-(SW2-A): track 42.8 -> 27.5 mm
- net Net-(Q2-S): track 0.00 -> 10.8 mm
- net Net-(U1-VC1): track 39.6 -> 29.4 mm
- net Net-(U1-ALERT): track 21.3 -> 31.3 mm
- net Net-(U1-VC0): track 30.8 -> 22.1 mm
- net Net-(U1-VC2): track 22.3 -> 14.8 mm
- net Net-(A1-A5/SCL): track 31.6 -> 37.3 mm
- net Net-(U1-VC5): track 20.4 -> 14.7 mm
- net Net-(Q1-G): track 53.2 -> 58.9 mm
- net Net-(U1-TS1): track 30.8 -> 35.7 mm
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Other:
- board size 96.5 x 99.1 mm -> 89.5 x 69.2 mm
- board text added: "2024"
- board text added: "BATT+"
- board text added: "BATT-"
- board text added: "Léon Becker"
- board text added: "PACK+"
- board text added: "PACK-"
- board text added: "The Ultimate Powerbank"
- board text added: "V1"

Commit message: Backup
Parts:
- C1, C2, C3, C6, C8: value 0.1μF -> 0.1uF
- C7, Cc1, Cc2, Cc3, Cc4: value 1μF -> 1uF
- C9: value 4.7μF -> 4.7uF
- Cf1: value 2.2μF -> 2.2uF
- R1, R3, Rf1: value 100Ω -> 100
- R2: value 8mΩ -> 8m
- R4: value 499kΩ -> 499k
- R5, R6, Rd1, Rd2: value 10kΩ -> 10k
- R7, R8: value 1MΩ -> 1M
- Rc1, Rc2, Rc3, Rc4: value 50Ω -> 50
Changed lines of the file:
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@@
 			)
 		)
-		(property "Value" "2.2μF"
+		(property "Value" "2.2uF"
 			(at 1.25 0 90)
 			(unlocked yes)
@@
 			)
 		)
-		(property "Value" "1MΩ"
+		(property "Value" "1M"
 			(at 5.842 0 0)
 			(unlocked yes)
@@
 		(fp_arc
 			(start 2.199991 3.050012)
-			(mid 2.141408 3.191422)
+			(mid 2.141406 3.191427)
 			(end 1.999991 3.250011)
 			(stroke
@@
 			)
 		)
-		(property "Value" "100Ω"
+		(property "Value" "100"
 			(at 6.096 0 180)
 			(unlocked yes)
@@
 			)
 		)
-		(property "Value" "1μF"
+		(property "Value" "1uF"
 			(at 2.5 0 -90)
 			(unlocked yes)
@@
 			)
 		)
-		(property "Value" "50Ω"
+		(property "Value" "50"
 			(at 6.477 0 0)
 			(unlocked yes)
@@
 			)
 		)
-		(property "Value" "499kΩ"
+		(property "Value" "499k"
 			(at 5.842 0 0)
 			(unlocked yes)
@@
 		)
 		(property "Mouser" "603-MFR-25FBF52-499K"
-			(at 0 0 360)
+			(at 0 0 0)
 			(layer "F.Fab")
 			(hide yes)
@@
 			)
 		)
-		(property "Value" "10kΩ"
+		(property "Value" "10k"
 			(at 3.937 0 0)
 			(unlocked yes)
@@
 			)
 		)
-		(property "Value" "50Ω"
+		(property "Value" "50"
 			(at 6.477 0 0)
 			(unlocked yes)
@@
 			)
 		)
-		(property "Value" "4.7μF"
+		(property "Value" "4.7uF"
 			(at 2.5 0 0)
 			(unlocked yes)
@@
 			)
 		)
-		(property "Value" "0.1μF"
+		(property "Value" "0.1uF"
 			(at 2.499995 0 0)
 			(unlocked yes)
@@
 			)
 		)
-		(property "Value" "1MΩ"
+		(property "Value" "1M"
 			(at 5.842 0 180)
 			(unlocked yes)
@@
 		(tags "Logo KiCad")
 		(property "Reference" "REF1"
-			(at 0 -5.08 360)
+			(at 0 -5.08 0)
 			(layer "F.SilkS")
 			(hide yes)
@@
 		)
 		(property "Value" "KiCad-Logo2_5mm_SilkScreen"
-			(at 0 5.08 360)
+			(at 0 5.08 0)
 			(layer "F.Fab")
 			(hide yes)
@@
 		)
 		(property "Mouser" "594-K471K10X7RF5UH5"
-			(at 0 0 270)
+			(at 0 0 -90)
 			(layer "F.Fab")
 			(hide yes)
@@
 			)
 		)
-		(property "Value" "10kΩ"
+		(property "Value" "10k"
 			(at 3.937 0 -90)
 			(unlocked yes)
@@
 			)
 		)
-		(property "Value" "1μF"
+		(property "Value" "1uF"
 			(at 2.5 0 -90)
 			(unlocked yes)
@@
 			)
 		)
-		(property "Value" "1μF"
+		(property "Value" "1uF"
 			(at 2.5 0 0)
 			(unlocked yes)
@@
 			)
 		)
+		(property ki_fp_filters "C_*")
+		(sheetname "Root")
+		(sheetfile "Powerbank.kicad_sch")
 		(attr through_hole)
 		(fp_line
@@
 			)
 		)
-		(property "Value" "10kΩ"
+		(property "Value" "10k"
 			(at 3.937 0 -90)
 			(unlocked yes)
@@
 			)
 		)
-		(property "Value" "100Ω"
+		(property "Value" "100"
 			(at 6.096 0 180)
 			(unlocked yes)
@@
 			)
 		)
-		(property "Value" "8mΩ"
+		(property "Value" "8m"
 			(at 12.192 0 0)
 			(unlocked yes)
@@
 			)
 		)
-		(property "Value" "0.1μF"
+		(property "Value" "0.1uF"
 			(at 2.499995 0 0)
 			(unlocked yes)
@@
 			)
 		)
-		(property "Value" "50Ω"
+		(property "Value" "50"
 			(at 6.477 0 0)
 			(unlocked yes)
@@
 			)
 		)
-		(property "Value" "10kΩ"
+		(property "Value" "10k"
 			(at 3.937 0 -90)
 			(unlocked yes)
@@
 			)
 		)
-		(property "Value" "50Ω"
+		(property "Value" "50"
 			(at 6.477 0 0)
 			(unlocked yes)
@@
 			)
 		)
-		(property "Value" "1μF"
+		(property "Value" "1uF"
 			(at 2.5 0 -90)
 			(unlocked yes)
@@
 			)
 		)
+		(property ki_fp_filters "C_*")
+		(sheetname "Root")
+		(sheetfile "Powerbank.kicad_sch")
 		(attr through_hole)
 		(fp_line
@@
 			)
 		)
-		(property "Value" "0.1μF"
+		(property "Value" "0.1uF"
 			(at 2.499995 0 0)
 			(unlocked yes)
@@
 			)
 		)
-		(property "Value" "0.1μF"
+		(property "Value" "0.1uF"
 			(at 2.499995 0 0)
 			(unlocked yes)
@@
 			)
 		)
-		(property "Value" "100Ω"
+		(property "Value" "100"
 			(at 6.096 0 -90)
 			(unlocked yes)
@@
 			)
 		)
-		(property "Value" "0.1μF"
+		(property "Value" "0.1uF"
 			(at 2.499995 0 90)
 			(unlocked yes)
@@
 		)
 		(property "Mouser" "594-K104K10X7RF53H5"
-			(at 0 0 270)
+			(at 0 0 -90)
 			(layer "F.Fab")
 			(hide yes)
@@
 			)
 		)
-		(property "Value" "1μF"
+		(property "Value" "1uF"
 			(at 2.5 0 -90)
 			(unlocked yes)

Commit message: Backup
Parts:
- added G***: LOGO, Symbol:Power bank symbol, F.Cu at (101.5, 89.4)
- moved G2 30.7 mm to (133.3, 96.5)
- moved R1 16.1 mm to (130.9, 113.5), turned to -90 degrees
- moved R3 11.0 mm to (134.7, 113.4), turned to -90 degrees
- moved Cc4 9.21 mm to (122.8, 119.4), turned to 90 degrees
- moved C1 7.76 mm to (127.5, 119.1), turned to 90 degrees
- moved C2 6.80 mm to (132.0, 111.1)
- moved D1 4.14 mm to (138.2, 84.6), turned to 180 degrees
- moved C3 3.92 mm to (138.2, 113.2), turned to -90 degrees
- moved G1 3.54 mm to (115.1, 119.6)
- moved Cc3 2.03 mm to (126.1, 106.6)
- moved C6 1.99 mm to (140.3, 134.6)
- moved C4 1.91 mm to (141.9, 117.5)
- moved R4 1.65 mm to (144.4, 116.1)
- moved R7 1.02 mm to (149.6, 124.5)
Routing:
- net GND: track 15.6 -> 35.4 mm
- net Net-(U1-SRP): track 30.9 -> 12.4 mm
- net Net-(U1-SRN): track 22.9 -> 11.9 mm
- net Net-(Q1-S): track 33.2 -> 24.4 mm
- net Net-(U1-VC0): track 22.1 -> 17.7 mm
- net Net-(C6-Pad2): track 1.80 -> 3.78 mm
- net Net-(U1-BAT): track 8.24 -> 6.30 mm
- net Net-(U1-VC1): track 29.4 -> 31.1 mm
- net Net-(D1-A): track 55.3 -> 53.9 mm
- net Net-(U1-TS1): track 35.7 -> 37.0 mm
- net Net-(D1-K): track 8.38 -> 7.26 mm
- net Net-(U1-ALERT): track 31.3 -> 30.3 mm
Other:
- board text added: "Do not touch!"
- board text added: "The Last Minute Life Saver"
- board text removed: "The Ultimate Powerbank"
