File: Circuit/KiCAD Circuit/Powerbank.kicad_pcb (KiCad board)
At the start: 2 copper layers, 89.5 x 69.2 mm, 50 parts, among them J1 EBWA-04-A, Q1 NMOS, Q2 PMOS, Q3 NMOS, SW1 SW_Push, SW2 SW_SPST, U1 BQ7692003PW

Commit message: Ordered
Other:
- rule pad_to_mask_clearance: 0.05 -> 0
Changed lines of the file:
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@@
 			(dielectric_constraints no)
 		)
-		(pad_to_mask_clearance 0.05)
+		(pad_to_mask_clearance 0)
 		(allow_soldermask_bridges_in_footprints no)
 		(pcbplotparams
@@
 			(plot_on_all_layers_selection 0x0000000_00000000)
 			(disableapertmacros no)
-			(usegerberextensions no)
-			(usegerberattributes yes)
-			(usegerberadvancedattributes yes)
-			(creategerberjobfile yes)
+			(usegerberextensions yes)
+			(usegerberattributes no)
+			(usegerberadvancedattributes no)
+			(creategerberjobfile no)
 			(dashed_line_dash_ratio 12.000000)
 			(dashed_line_gap_ratio 3.000000)
@@
 			(psa4output no)
 			(plotreference yes)
-			(plotvalue yes)
+			(plotvalue no)
 			(plotfptext yes)
 			(plotinvisibletext no)
 			(sketchpadsonfab no)
-			(subtractmaskfromsilk no)
+			(subtractmaskfromsilk yes)
 			(outputformat 1)
 			(mirror no)
-			(drillshape 1)
+			(drillshape 0)
 			(scaleselection 1)
-			(outputdirectory "")
+			(outputdirectory "Fabrication Files/")
 		)
 	)
@@
 		(fp_arc
 			(start 2.199991 3.050012)
-			(mid 2.141408 3.191422)
+			(mid 2.141406 3.191427)
 			(end 1.999991 3.250011)
 			(stroke
@@
 		)
 		(property "Mouser" "603-MFR-25FBF52-499K"
-			(at 0 0 360)
+			(at 0 0 0)
 			(layer "F.Fab")
 			(hide yes)
@@
 				(font
 					(size 1.27 1.27)
-					(thickness 0.35)
+					(thickness 0.3175)
 				)
 			)
@@
 		(tags "net tie")
 		(property "Reference" "NT2"
-			(at 0 -1.2 270)
+			(at 0 -1.2 -90)
 			(layer "F.SilkS")
 			(hide yes)
@@
 		)
 		(property "Value" "NetTie"
-			(at 0 1.2 270)
+			(at 0 1.2 -90)
 			(layer "F.Fab")
 			(hide yes)
