File: Circuit/KiCAD Circuit/Powerbank.kicad_sch (KiCad schematic)
At the start: 45 parts, among them Q1 NMOS, Q2 PMOS, Q3 NMOS, SW1 SW_Push, SW2 SW_SPST, U1 BQ7692003PWR, U2 Arduino_Nano_v3.x, U3 AZ1117CH-5.0TRG1

Commit message: Backup
Other:
- removed sheet MAX1758
Changed lines of the file:
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@@
   (symbol (lib_id "power:GND") (at 213.36 72.39 0) (unit 1)
     (in_bom yes) (on_board yes) (dnp no) (fields_autoplaced)
-    (property "Reference" "#PWR027" (at 213.36 78.74 0)
+    (property "Reference" "#PWR012" (at 213.36 78.74 0)
       (effects (font (size 1.27 1.27)) hide)
     )
@@
       (project "Powerbank"
         (path "/b34928fe-f013-4cc5-8c95-edbe1f5c3ffc"
-          (reference "#PWR027") (unit 1)
+          (reference "#PWR012") (unit 1)
         )
       )
@@
   (symbol (lib_id "power:GND") (at 71.755 147.955 0) (unit 1)
     (in_bom yes) (on_board yes) (dnp no) (fields_autoplaced)
-    (property "Reference" "#PWR07" (at 71.755 154.305 0)
+    (property "Reference" "#PWR01" (at 71.755 154.305 0)
       (effects (font (size 1.27 1.27)) hide)
     )
@@
       (project "Powerbank"
         (path "/b34928fe-f013-4cc5-8c95-edbe1f5c3ffc"
-          (reference "#PWR07") (unit 1)
+          (reference "#PWR01") (unit 1)
         )
       )
@@
   (symbol (lib_id "power:GND") (at 116.84 137.16 0) (unit 1)
     (in_bom yes) (on_board yes) (dnp no) (fields_autoplaced)
-    (property "Reference" "#PWR019" (at 116.84 143.51 0)
+    (property "Reference" "#PWR05" (at 116.84 143.51 0)
       (effects (font (size 1.27 1.27)) hide)
     )
@@
       (project "Powerbank"
         (path "/b34928fe-f013-4cc5-8c95-edbe1f5c3ffc"
-          (reference "#PWR019") (unit 1)
+          (reference "#PWR05") (unit 1)
         )
       )
@@
   (symbol (lib_id "power:GND") (at 149.86 98.425 0) (unit 1)
     (in_bom yes) (on_board yes) (dnp no) (fields_autoplaced)
-    (property "Reference" "#PWR025" (at 149.86 104.775 0)
+    (property "Reference" "#PWR010" (at 149.86 104.775 0)
       (effects (font (size 1.27 1.27)) hide)
     )
@@
       (project "Powerbank"
         (path "/b34928fe-f013-4cc5-8c95-edbe1f5c3ffc"
-          (reference "#PWR025") (unit 1)
+          (reference "#PWR010") (unit 1)
         )
       )
@@
   (symbol (lib_id "power:GNDREF") (at 73.66 133.35 0) (unit 1)
     (in_bom yes) (on_board yes) (dnp no) (fields_autoplaced)
-    (property "Reference" "#PWR016" (at 73.66 139.7 0)
+    (property "Reference" "#PWR02" (at 73.66 139.7 0)
       (effects (font (size 1.27 1.27)) hide)
     )
@@
       (project "Powerbank"
         (path "/b34928fe-f013-4cc5-8c95-edbe1f5c3ffc"
-          (reference "#PWR016") (unit 1)
+          (reference "#PWR02") (unit 1)
         )
       )
@@
   (symbol (lib_id "power:GND") (at 161.29 98.425 0) (unit 1)
     (in_bom yes) (on_board yes) (dnp no) (fields_autoplaced)
-    (property "Reference" "#PWR026" (at 161.29 104.775 0)
+    (property "Reference" "#PWR011" (at 161.29 104.775 0)
       (effects (font (size 1.27 1.27)) hide)
     )
@@
       (project "Powerbank"
         (path "/b34928fe-f013-4cc5-8c95-edbe1f5c3ffc"
-          (reference "#PWR026") (unit 1)
+          (reference "#PWR011") (unit 1)
         )
       )
@@
   (symbol (lib_id "power:GND") (at 88.9 100.33 0) (unit 1)
     (in_bom yes) (on_board yes) (dnp no) (fields_autoplaced)
-    (property "Reference" "#PWR017" (at 88.9 106.68 0)
+    (property "Reference" "#PWR03" (at 88.9 106.68 0)
       (effects (font (size 1.27 1.27)) hide)
     )
@@
       (project "Powerbank"
         (path "/b34928fe-f013-4cc5-8c95-edbe1f5c3ffc"
-          (reference "#PWR017") (unit 1)
+          (reference "#PWR03") (unit 1)
         )
       )
@@
   (symbol (lib_id "power:GNDREF") (at 101.6 133.35 0) (unit 1)
     (in_bom yes) (on_board yes) (dnp no) (fields_autoplaced)
-    (property "Reference" "#PWR018" (at 101.6 139.7 0)
+    (property "Reference" "#PWR04" (at 101.6 139.7 0)
       (effects (font (size 1.27 1.27)) hide)
     )
@@
       (project "Powerbank"
         (path "/b34928fe-f013-4cc5-8c95-edbe1f5c3ffc"
-          (reference "#PWR018") (unit 1)
+          (reference "#PWR04") (unit 1)
         )
       )
@@
   (symbol (lib_id "power:GND") (at 260.35 72.39 0) (unit 1)
     (in_bom yes) (on_board yes) (dnp no) (fields_autoplaced)
-    (property "Reference" "#PWR029" (at 260.35 78.74 0)
+    (property "Reference" "#PWR014" (at 260.35 78.74 0)
       (effects (font (size 1.27 1.27)) hide)
     )
@@
       (project "Powerbank"
         (path "/b34928fe-f013-4cc5-8c95-edbe1f5c3ffc"
-          (reference "#PWR029") (unit 1)
+          (reference "#PWR014") (unit 1)
         )
       )
@@
   (symbol (lib_id "power:GND") (at 139.7 98.425 0) (unit 1)
     (in_bom yes) (on_board yes) (dnp no) (fields_autoplaced)
-    (property "Reference" "#PWR022" (at 139.7 104.775 0)
+    (property "Reference" "#PWR08" (at 139.7 104.775 0)
       (effects (font (size 1.27 1.27)) hide)
     )
@@
       (project "Powerbank"
         (path "/b34928fe-f013-4cc5-8c95-edbe1f5c3ffc"
-          (reference "#PWR022") (unit 1)
+          (reference "#PWR08") (unit 1)
         )
       )
@@
   (symbol (lib_id "power:GND") (at 127 71.755 0) (unit 1)
     (in_bom yes) (on_board yes) (dnp no) (fields_autoplaced)
-    (property "Reference" "#PWR020" (at 127 78.105 0)
+    (property "Reference" "#PWR06" (at 127 78.105 0)
       (effects (font (size 1.27 1.27)) hide)
     )
@@
       (project "Powerbank"
         (path "/b34928fe-f013-4cc5-8c95-edbe1f5c3ffc"
-          (reference "#PWR020") (unit 1)
+          (reference "#PWR06") (unit 1)
         )
       )
@@
   (symbol (lib_id "power:GND") (at 131.445 121.285 0) (unit 1)
     (in_bom yes) (on_board yes) (dnp no) (fields_autoplaced)
-    (property "Reference" "#PWR021" (at 131.445 127.635 0)
+    (property "Reference" "#PWR07" (at 131.445 127.635 0)
       (effects (font (size 1.27 1.27)) hide)
     )
@@
       (project "Powerbank"
         (path "/b34928fe-f013-4cc5-8c95-edbe1f5c3ffc"
-          (reference "#PWR021") (unit 1)
+          (reference "#PWR07") (unit 1)
         )
       )
@@
   (symbol (lib_id "power:GND") (at 227.33 130.81 0) (unit 1)
     (in_bom yes) (on_board yes) (dnp no) (fields_autoplaced)
-    (property "Reference" "#PWR028" (at 227.33 137.16 0)
+    (property "Reference" "#PWR013" (at 227.33 137.16 0)
       (effects (font (size 1.27 1.27)) hide)
     )
@@
       (project "Powerbank"
         (path "/b34928fe-f013-4cc5-8c95-edbe1f5c3ffc"
-          (reference "#PWR028") (unit 1)
+          (reference "#PWR013") (unit 1)
         )
       )
@@
   (symbol (lib_id "power:GNDREF") (at 147.955 118.11 0) (unit 1)
     (in_bom yes) (on_board yes) (dnp no) (fields_autoplaced)
-    (property "Reference" "#PWR023" (at 147.955 124.46 0)
+    (property "Reference" "#PWR09" (at 147.955 124.46 0)
       (effects (font (size 1.27 1.27)) hide)
     )
@@
       (project "Powerbank"
         (path "/b34928fe-f013-4cc5-8c95-edbe1f5c3ffc"
-          (reference "#PWR023") (unit 1)
+          (reference "#PWR09") (unit 1)
         )
       )
@@
       )
     )
-  )
-  (sheet (at 21.59 20.32) (size 12.7 5.08) (fields_autoplaced)
-    (stroke (width 0.1524) (type solid))
-    (fill (color 0 0 0 0.0000))
-    (property "Sheetname" "MAX1758" (at 21.59 19.6084 0)
-      (effects (font (size 1.27 1.27)) (justify left bottom))
-    )
-    (property "Sheetfile" "MAX1758.kicad_sch" (at 21.59 25.9846 0)
-      (effects (font (size 1.27 1.27)) (justify left top))
-    )
-    (instances
-      (project "Powerbank"
-        (path "/b34928fe-f013-4cc5-8c95-edbe1f5c3ffc" (page "2"))
-      )
-    )

Commit message: Backup
Parts:
- removed C12: 22μF, symbol Device:C_Small
- removed C13: 10μF, symbol Device:C_Small
- removed U1: BQ7692003PWR, PW0020A_N, symbol BQ2692006PWR:BQ7692006PWR
- removed U3: AZ1117CH-5.0TRG1, SOT-223_DIO, symbol AZ1117CH-5.0TRG1:AZ1117CH-5.0TRG1
- added D2: D, symbol Device:D
- added Rd2: 10kΩ, RNF18FTD10K0:STA_RNF18_STP, symbol Device:R_US
- added U1: BQ7692003PW, BQ7692003PW:PW0020A_N, symbol BQ7692003PW:BQ7692003PW
- C1, C10, C11, C2, C3, C6, C8: footprint (none) -> K104K10X7RF53H5:K104K10X7RF53H5_VIS; Mouser (none) -> 594-K104K10X7RF53H5
- C4: footprint (none) -> K471K10X7RF5UH5:K471K10X7RF5UH5_VIS; Mouser (none) -> 594-K471K10X7RF5UH5
- C5: footprint (none) -> C410C472K1R5TA:CAP_C410C_AX_X7R_AXIMAX_KEM; Mouser (none) -> 80-C410C472K1R
- C7, Cc1, Cc2, Cc3, Cc4: footprint (none) -> K105K20X7RF5TH5:K105K20X7RF5TH5_VIS; Mouser (none) -> K105K20X7RF5TH5
- C9: footprint (none) -> FG24X7R1E475KRT06:CAP_FG24_TDK; Mouser (none) -> 810-FG24X7R1E475KRT6
- Cf1: footprint (none) -> FG18X5R1E225KRT06:CAP_FG18_TDK; Mouser (none) -> 810-FG18X5R1E225KRT6
- D3: renamed from D2; value D_TVS_uni -> TVS Diode 17.1V; footprint (none) -> Diode_THT:D_DO-41_SOD81_P7.62mm_Horizontal; Mouser (none) -> 576-P4KE20A
- Q1, Q3: footprint (none) -> Custom Footprints:TO-220AB; Mouser (none) -> 942-IRLB4132PBF
- R1, R3, Rf1: footprint (none) -> RNF14FTD100R:STA_RNF14_STP; Mouser (none) -> 708-RNF14FTD100R
- R2: footprint (none) -> 14AFR008E:RES_14A_OHM; Mouser (none) -> 588-14AFR008E
- R4: value 500kΩ -> 499kΩ; footprint (none) -> MFR-25FBF52-499K:YAG_MF25_YAG; Mouser (none) -> 603-MFR-25FBF52-499K
- R5, R6, Rd1: footprint (none) -> RNF18FTD10K0:STA_RNF18_STP; Mouser (none) -> 708-RNF18FTD10K0
- R7, R8: footprint (none) -> MFR-25FRF52-1M:YAG_MF25_YAG; Mouser (none) -> 603-MFR-25FRF521M
- Rc1, Rc2, Rc3, Rc4: footprint (none) -> CMF5550R000FKEK70:RES_CMF07_VIS; Mouser (none) -> CMF5550R000FKEK70
- SW1, SW2: footprint (none) -> Custom Footprints:Push button; Details (none) -> Using item from home stock.
- U2: footprint Module:Arduino_Nano -> Arduinos:Arduino_Nano_33_IoT_Socket
Connections:
- net GNDREF is gone; now on net GND: C1.1, C3.2, Q2.2 (G)
- net GND: now also U1.3 (VSS)
- net PACK +: now also D2.2 (A), Rd2.1; no longer SW2.1 (A)
- net at Q1.2 (G), R7.1: now also U1.1 (DSG)
- net at Cf1.1, Rf1.2: now also U1.10 (BAT), U1.9 (REGSRC)
- net at Cc1.1, Rc1.2: now also U1.12 (VC5)
- net at Cc1.2, Cc2.1, Rc2.2: now also U1.13 (VC4), U1.14 (VC3), U1.15 (VC2)
- net at Cc2.2, Cc3.1, Rc3.2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: now also U1.16 (VC1)
- net at Cc4.2, Rc4.2: now also U1.17 (VC0)
- net at C1.2, C2.1, R1.1: now also U1.18 (SRP)
- net at C2.2, C3.1, R3.1: now also U1.19 (SRN)
- net at Q2.3 (S): now also U1.2 (CHG)
- net at C4.2, R4.1, U2.13 (D10): now also U1.20 (ALERT)
- net at U2.23 (A4_SDA): now also U1.4 (SDA)
- net at U2.24 (A5_SCL): now also U1.5 (SCL)
- net at C5.1, R5.2, R6.1: now also U1.6 (TS1)
- net at C7.1: now also U1.7 (CAP1)
- net at C9.1: now also U1.8 (REGOUT)
- net at U2.30 (VIN): now also SW2.1 (A)
- net at SW2.2 (B): now also D2.1 (K), Rd2.2
- no-connect marks 0 -> 25
Other:
- moved on the sheet: C1, C10, C11, C2, C3, C4, C5, C6, C7, C8, C9, CELL_1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

Commit message: Backup
Parts:
- removed C10, C11: 0.1μF, K104K10X7RF53H5:K104K10X7RF53H5_VIS, symbol Device:C_Small
- removed CELL_1, CELL_2, CELL_3: ~, symbol Device:Battery_Cell
- removed U2: Arduino_Nano_v3.x, Arduinos:Arduino_Nano_33_IoT_Socket, symbol MCU_Module:Arduino_Nano_v3.x
- added A1: Arduino_Nano_33_IoT_Socket, Arduinos:Arduino_Nano_33_IoT_Socket, symbol Arduinos:Arduino_Nano_33_IoT_Socket
- added H1: BATT+, Custom Footprints:Power Connection Pads, symbol Mechanical:MountingHole_Pad
- added H2: BATT-, Custom Footprints:Power Connection Pads, symbol Mechanical:MountingHole_Pad
- added H7: PACK+, Custom Footprints:Power Connection Pads, symbol Mechanical:MountingHole_Pad
- added H8: PACK-, Custom Footprints:Power Connection Pads, symbol Mechanical:MountingHole_Pad
- added J1: EBWA-04-A, Custom Footprints:EBWA-04-A, symbol EBWA-04-A:EBWA-04-A
- D1, D2: footprint (none) -> Custom Footprints:1N4149TR; Mouser (none) -> 512-1N4149TR
- Q1, Q3: footprint Custom Footprints:TO-220AB -> Custom Footprints:IRLB4132PBF
- Q2: footprint (none) -> VP3203N3-G:TO-92_MC_MCH; Mouser (none) -> 689-VP3203N3-G
- Rc1, Rc2, Rc3, Rc4: Mouser CMF5550R000FKEK70 -> 71-CMF5550R000FKEK70
- SW1, SW2: footprint Custom Footprints:Push button -> Custom Footprints:Switch Pads
Connections:
- net GND: now also D3.2 (A), A1.GND1 (GND), A1.GND2 (GND), H2.1, J1.1 (C0)
- net at Rc2.1: now also J1.3 (C2)
- net at Rc3.1: now also J1.2 (C1)
- net at C4.2, R4.1, U1.20 (ALERT): now also A1.D10
- net at SW2.1 (A): now also A1.VIN
- net at U1.4 (SDA): now also A1.A4 (A4/SDA)
- net at U1.5 (SCL): now also A1.A5 (A5/SCL)
- net PACK +: no longer names the net of D1.2 (A), D2.2 (A), D3.1 (K), Rc1.1, Rd1.1, Rd2.1
- net PACK +: now also H1.1, H7.1, J1.4 (C5)
- net PACK -: no longer names the net of C8.2, Q3.3 (S), R8.2
- net PACK -: now also H8.1; no longer D3.2 (A)
- no-connect marks 25 -> 24
Other:
- moved on the sheet: D3

Commit message: Backup
Other:
- note added: "Measurement: single cell voltages, pack voltage, coulomb counter, die thermistor, receive ALERT signal Protection: over-voltage (OV), under-voltage (UV), over-current in discharge (OCD), short-circuit in discharge (SCD) Control: CHG, DSG, cell balancing, sent ALERT signal"
- company: [Private] Léon Becker -> Léon Becker
- title: BQ76920 Power Bank Circuit -> BQ76920 Power Bank Schematic
- moved on the sheet: A1, C2, C4, C5, C6, D1, D2, H1, H2, H7, H8, J1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

Commit message: Backup
Parts:
- added NT1, NT2: NetTie, Custom Footprints:NetTie General Net Class, symbol Device:NetTie_2
- C7: Mouser K105K20X7RF5TH5 -> 594-K105K20X7RF5TH5
- Q2: footprint VP3203N3-G:TO-92_MC_MCH -> Custom Footprints:TO-92_MC_MCH
Connections:
- net GND: now also NT2.1; no longer U1.3 (VSS)
- net at D3.1 (K), H1.1, H7.1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: now also NT1.1; no longer D1.2 (A), D2.2 (A), Rd1.1, Rd2.1
- new net: D1.2 (A), D2.2 (A), NT1.2, Rd1.1, Rd2.1
- new net: NT2.2, U1.3 (VSS)
Other:
- moved on the sheet: Q1, R7

Commit message: Backup
Parts:
- C1, C2, C3, C6, C8: value 0.1μF -> 0.1uF
- C7, Cc1, Cc2, Cc3, Cc4: value 1μF -> 1uF
- C9: value 4.7μF -> 4.7uF
- Cf1: value 2.2μF -> 2.2uF
- R1, R3, Rf1: value 100Ω -> 100
- R2: value 8mΩ -> 8m
- R4: value 499kΩ -> 499k
- R5, R6, Rd1, Rd2: value 10kΩ -> 10k
- R7, R8: value 1MΩ -> 1M
- Rc1, Rc2, Rc3, Rc4: value 50Ω -> 50
Changed lines of the file:
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@@
 			)
 		)
-		(property "Value" "0.1μF"
+		(property "Value" "0.1uF"
 			(at 84.455 121.92 90)
 			(effects
@@
 		(fields_autoplaced yes)
 		(property "Reference" "Cf1"
-			(at 135.89 83.8263 0)
+			(at 135.89 83.8262 0)
 			(effects
 				(font
@@
 			)
 		)
-		(property "Value" "2.2μF"
-			(at 135.89 86.3663 0)
+		(property "Value" "2.2uF"
+			(at 135.89 86.3662 0)
 			(effects
 				(font
@@
 			)
 		)
-		(property "Value" "100Ω"
+		(property "Value" "100"
 			(at 59.69 129.54 0)
 			(effects
@@
 		(fields_autoplaced yes)
 		(property "Reference" "C9"
-			(at 147.32 83.8263 0)
+			(at 147.32 83.8262 0)
 			(effects
 				(font
@@
 			)
 		)
-		(property "Value" "4.7μF"
-			(at 147.32 86.3663 0)
+		(property "Value" "4.7uF"
+			(at 147.32 86.3662 0)
 			(effects
 				(font
@@
 			)
 		)
-		(property "Value" "50Ω"
+		(property "Value" "50"
 			(at 71.12 95.25 90)
 			(effects
@@
 			)
 		)
-		(property "Value" "1μF"
+		(property "Value" "1uF"
 			(at 79.375 74.93 0)
 			(effects
@@
 			)
 		)
-		(property "Value" "0.1μF"
+		(property "Value" "0.1uF"
 			(at 120.65 146.685 90)
 			(effects
@@
 		(on_board yes)
 		(dnp no)
-		(fields_autoplaced yes)
 		(property "Reference" "R6"
-			(at 103.505 55.88 0)
+			(at 104.14 55.88 0)
 			(effects
 				(font
@@
 			)
 		)
-		(property "Value" "10kΩ"
-			(at 103.505 58.42 0)
+		(property "Value" "10k"
+			(at 104.14 58.42 0)
 			(effects
 				(font
@@
 			)
 		)
-		(property "Value" "499kΩ"
+		(property "Value" "499k"
 			(at 102.87 123.19 0)
 			(effects
@@
 			)
 		)
-		(property "Value" "1μF"
+		(property "Value" "1uF"
 			(at 79.375 82.55 0)
 			(effects
@@
 			)
 		)
-		(property "Value" "100Ω"
+		(property "Value" "100"
 			(at 80.01 129.54 0)
 			(effects
@@
 		(fields_autoplaced yes)
 		(property "Reference" "Rd1"
-			(at 136.525 49.53 0)
+			(at 137.16 49.5299 0)
 			(effects
 				(font
@@
 			)
 		)
-		(property "Value" "10kΩ"
-			(at 136.525 52.07 0)
+		(property "Value" "10k"
+			(at 137.16 52.0699 0)
 			(effects
 				(font
@@
 			)
 		)
-		(property "Value" "0.1μF"
+		(property "Value" "0.1uF"
 			(at 133.3563 146.05 90)
 			(effects
@@
 		(fields_autoplaced yes)
 		(property "Reference" "Rf1"
-			(at 127.635 59.69 0)
+			(at 128.27 59.6899 0)
 			(effects
 				(font
@@
 			)
 		)
-		(property "Value" "100Ω"
-			(at 127.635 62.23 0)
+		(property "Value" "100"
+			(at 128.27 62.2299 0)
 			(effects
 				(font
@@
 			)
 		)
-		(property "Value" "10kΩ"
+		(property "Value" "10k"
 			(at 180.34 52.07 0)
 			(effects
@@
 			)
 		)
-		(property "Value" "1μF"
+		(property "Value" "1uF"
 			(at 79.375 93.98 0)
 			(effects
@@
 			)
 		)
-		(property "Value" "50Ω"
+		(property "Value" "50"
 			(at 71.755 76.2 90)
 			(effects
@@
 			)
 		)
-		(property "Value" "50Ω"
+		(property "Value" "50"
 			(at 71.755 83.82 90)
 			(effects
@@
 			)
 		)
-		(property "Value" "1MΩ"
+		(property "Value" "1M"
 			(at 144.78 131.445 0)
 			(effects
@@
 			)
 		)
-		(property "Value" "0.1μF"
+		(property "Value" "0.1uF"
 			(at 72.39 120.015 90)
 			(effects
@@
 		(fields_autoplaced yes)
 		(property "Reference" "C7"
-			(at 125.73 83.8263 0)
+			(at 125.73 83.8262 0)
 			(effects
 				(font
@@
 			)
 		)
-		(property "Value" "1μF"
-			(at 125.73 86.3663 0)
+		(property "Value" "1uF"
+			(at 125.73 86.3662 0)
 			(effects
 				(font
@@
 		(on_board yes)
 		(dnp no)
-		(fields_autoplaced yes)
 		(property "Reference" "Rc1"
-			(at 63.5 68.58 90)
+			(at 62.23 68.58 90)
 			(effects
 				(font
@@
 			)
 		)
-		(property "Value" "50Ω"
-			(at 71.755 68.58 90)
+		(property "Value" "50"
+			(at 71.12 68.58 90)
 			(effects
 				(font
@@
 			)
 		)
-		(property "Value" "1MΩ"
+		(property "Value" "1M"
 			(at 106.68 132.08 0)
 			(effects
@@
 			)
 		)
-		(property "Value" "1μF"
+		(property "Value" "1uF"
 			(at 79.375 88.9 0)
 			(effects
@@
 			)
 		)
-		(property "Value" "10kΩ"
+		(property "Value" "10k"
 			(at 106.68 48.26 90)
 			(effects
@@
 			)
 		)
-		(property "Value" "0.1μF"
+		(property "Value" "0.1uF"
 			(at 64.135 121.92 90)
 			(effects
@@
 			)
 		)
-		(property "Value" "8mΩ"
+		(property "Value" "8m"
 			(at 72.39 140.335 90)
 			(effects

Commit message: Backup
Parts:
- D1, D2: Mouser 512-1N4149TR -> 512-1N4149
Changed lines of the file:
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@@
 			)
 		)
-		(property "Mouser" "512-1N4149TR"
+		(property "Mouser" "512-1N4149"
 			(at 170.18 50.8 90)
 			(effects
@@
 			)
 		)
-		(property "Mouser" "512-1N4149TR"
+		(property "Mouser" "512-1N4149"
 			(at 125.73 50.8 90)
 			(effects

Commit message: Ordered
Parts:
- Cc1, Cc2, Cc3, Cc4: Mouser K105K20X7RF5TH5 -> 594-K105K20X7RF5TH5
